Commit message: Set up the rest of the launch files and gazebo components

File: kohm_description/urdf/kohm.urdf (robot description, URDF)
Before this commit: robot kohm, 12 links, 11 joints
Links:
- removed link Camera_Link
- removed link Caster_Wheel
- removed link Front_Mast_Pillar
- removed link Imu_Link
- removed link Left_Front_Wheel
- removed link Lidar_Link
- removed link Mid_Mast_Pillar
- removed link Rear_Mast_Pillar
- removed link Right_Front_Wheel
- removed link Top_Mast_Pillar
- added link camera_link, mass 0.1; collision box size=0.0508 0.0508 0.1016; visual box size=0.1016 0.0508 0.0508
- added link caster_wheel, mass 2; collision sphere radius=0.165; visual sphere radius=0.1651
- added link front_mast_pillar, mass 1; collision box size=0.0254 0.0254 1.2954; visual box size=0.0254 0.0254 1.2954
- added link imu_link, mass 1; collision box size=0.0254 0.0254 0.0254; visual box size=0.0254 0.0254 0.0254
- added link laser_link, mass 1; collision cylinder length=0.1524 radius=0.0762; visual cylinder length=0.1524 radius=0.0762
- added link left_front_wheel, mass 2.25; collision cylinder length=0.1 radius=0.165; visual cylinder length=0.1 radius=0.165
- added link mid_mast_pillar, mass 1; collision box size=0.0254 0.0254 1.2954; visual box size=0.4064 0.0254 0.0254
- added link rear_mast_pillar, mass 1; collision box size=0.0254 0.0254 1.2954; visual box size=0.0254 0.0254 1.2954
- added link right_front_wheel, mass 2.25; collision cylinder length=0.1 radius=0.165; visual cylinder length=0.1 radius=0.165
- added link top_mast_pillar, mass 1; collision box size=1.016 0.0254 0.0254; visual box size=1.016 0.0254 0.0254
Joints:
- removed joint Camera_Link_to_base_link
- removed joint Caster_Wheel_to_base_link
- removed joint Front_Mast_Pillar_to_base_link
- removed joint Imu_Link_to_base_link
- removed joint Left_Front_Wheel_to_Base_Link
- removed joint Lidar_to_base_link
- removed joint Mid_Mast_Pillar_to_base_link
- removed joint Rear_Mast_Pillar_to_base_link
- removed joint Right_Front_Wheel_to_Base_Link
- removed joint Top_Mast_Pillar_to_base_link
- added joint camera_link_to_base_link: type fixed, parent base_link, child camera_link, origin xyz=0.3992 0 1.3716 rpy=0 0.785398 0
- added joint caster_wheel_to_base_link: type fixed, parent base_link, child caster_wheel, origin xyz=-0.285 0 -0.0508 rpy=0 0 0
- added joint front_mast_pillar_to_base_link: type fixed, parent base_link, child front_mast_pillar, origin xyz=0.1833 0 0.7747 rpy=0 0 0
- added joint imu_link_to_base_link: type fixed, parent base_link, child imu_link, origin xyz=-0.012 0 0.5588 rpy=0 0 0
- added joint laser_to_base_link: type fixed, parent base_link, child laser_link, origin xyz=0.2722 0 0.3556 rpy=0 0 0
- added joint left_front_wheel_to_base_link: type continuous, parent base_link, child left_front_wheel, origin xyz=0.285 0.27 -0.0508 rpy=0 0 0, axis 0 1 0
- added joint mid_mast_pillar_to_base_link: type fixed, parent base_link, child mid_mast_pillar, origin xyz=-0.012 0 0.5461 rpy=0 0 0
- added joint rear_mast_pillar_to_base_link: type fixed, parent base_link, child rear_mast_pillar, origin xyz=-0.223 0 0.7747 rpy=0 0 0
- added joint right_front_wheel_to_base_link: type continuous, parent base_link, child right_front_wheel, origin xyz=0.285 -0.27 -0.0508 rpy=0 0 0, axis 0 1 0
- added joint top_mast_pillar_to_base_link: type fixed, parent base_link, child top_mast_pillar, origin xyz=-0.012 0 1.4224 rpy=0 0 0

Commit message: Added 3x the wheels to kohm

File: kohm_description/urdf/kohm.urdf (robot description, URDF)
Before this commit: robot kohm, 12 links, 11 joints
Links:
- removed link caster_wheel
- added link left_mid_wheel, mass 2.25; collision cylinder length=0.1 radius=0.165; visual cylinder length=0.1 radius=0.165
- added link left_rear_wheel, mass 2.25; collision cylinder length=0.1 radius=0.165; visual cylinder length=0.1 radius=0.165
- added link right_mid_wheel, mass 2.25; collision cylinder length=0.1 radius=0.165; visual cylinder length=0.1 radius=0.165
- added link right_rear_wheel, mass 2.25; collision cylinder length=0.1 radius=0.165; visual cylinder length=0.1 radius=0.165
Joints:
- removed joint caster_wheel_to_base_link
- added joint left_mid_wheel_to_base_link: type continuous, parent base_link, child left_mid_wheel, origin xyz=0 0.27 -0.0508 rpy=0 0 0, axis 0 1 0
- added joint left_rear_wheel_to_base_link: type continuous, parent base_link, child left_rear_wheel, origin xyz=-0.285 0.27 -0.0508 rpy=0 0 0, axis 0 1 0
- added joint right_mid_wheel_to_base_link: type continuous, parent base_link, child right_mid_wheel, origin xyz=0 -0.27 -0.0508 rpy=0 0 0, axis 0 1 0
- added joint right_rear_wheel_to_base_link: type continuous, parent base_link, child right_rear_wheel, origin xyz=-0.285 -0.27 -0.0508 rpy=0 0 0, axis 0 1 0

Commit message: Rotate camera lmao

File: kohm_description/urdf/kohm.urdf (robot description, URDF)
Before this commit: robot kohm, 15 links, 14 joints
Joints:
- joint camera_link_to_base_link: origin xyz=0.3992 0 1.3716 rpy=0 0.785398 0 -> xyz=0.3992 0 1.3716 rpy=0 0.872665 0

File: kohm_description/urdf/kohm_robot.urdf (robot description, URDF)
Before this commit: robot kohm, 15 links, 14 joints
Joints:
- joint camera_link_to_base_link: origin xyz=0.3992 0 1.3716 rpy=0 0.785398 0 -> xyz=0.3992 0 1.3716 rpy=0 0.872665 0

Commit message: add potential wld angle

File: kohm_description/urdf/kohm.urdf (robot description, URDF)
Before this commit: robot kohm, 15 links, 14 joints
Joints:
- joint camera_link_to_base_link: origin xyz=0.3992 0 1.3716 rpy=0 0.872665 0 -> xyz=0.3992 0 1.3716 rpy=0 0.785398 0
