Commit message: avery changes lmao

File: kohm_description/urdf/kohm_robot.urdf (robot description, URDF)
Before this commit: robot kohm, 15 links, 14 joints
Joints:
- joint laser_to_base_link: origin xyz=0.2722 0 0.3556 rpy=0 0 0 -> xyz=0.2722 0 0.3556 rpy=0 0 3.14

Commit message: galactic update BABY

File: kohm_description/urdf/kohm_robot.urdf (robot description, URDF)
Before this commit: robot kohm, 15 links, 14 joints
Joints:
- joint laser_to_base_link: origin xyz=0.2722 0 0.3556 rpy=0 0 3.14 -> xyz=0.2722 0 0.3556 rpy=0 0 0

Commit message: Moved base footprint back so that the kohm's pivot point is closer to irl

File: kohm_description/urdf/kohm_robot.urdf (robot description, URDF)
Before this commit: robot kohm, 15 links, 14 joints
Joints:
- joint base_footprint_to_base_link: origin xyz=0 0 0.225 rpy=0 0 0 -> xyz=0.285 0 0.225 rpy=0 0 0
